File: PCB_Design/Titan-Legs/CAN_BUS.kicad_sch (KiCad schematic)
At the start: 4 parts

Commit message: schematics 1st iteration completed
Parts:
- gave numbers to parts that had none: 4
Changed lines of the file:
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@@
   (symbol (lib_id "power:GND") (at 170.18 105.41 0) (unit 1)
     (in_bom yes) (on_board yes)
-    (property "Reference" "#PWR?" (id 0) (at 170.18 111.76 0)
+    (property "Reference" "#PWR025" (id 0) (at 170.18 111.76 0)
       (effects (font (size 1.27 1.27)) hide)
     )
@@
   (symbol (lib_id "power:GND") (at 152.4 110.49 0) (unit 1)
     (in_bom yes) (on_board yes) (fields_autoplaced)
-    (property "Reference" "#PWR?" (id 0) (at 152.4 116.84 0)
+    (property "Reference" "#PWR024" (id 0) (at 152.4 116.84 0)
       (effects (font (size 1.27 1.27)) hide)
     )
@@
   (symbol (lib_id "Device:C") (at 170.18 99.06 0) (unit 1)
     (in_bom yes) (on_board yes)
-    (property "Reference" "C?" (id 0) (at 171.45 96.52 0)
+    (property "Reference" "C9" (id 0) (at 171.45 96.52 0)
       (effects (font (size 1 1)) (justify left))
     )
@@
   (symbol (lib_id "Device:R") (at 110.49 102.87 0) (unit 1)
     (in_bom yes) (on_board yes)
-    (property "Reference" "R?" (id 0) (at 113.03 100.33 0)
+    (property "Reference" "R13" (id 0) (at 113.03 100.33 0)
       (effects (font (size 1 1)) (justify left))
     )
@@
   (symbol (lib_id "power:GND") (at 110.49 107.95 0) (unit 1)
     (in_bom yes) (on_board yes) (fields_autoplaced)
-    (property "Reference" "#PWR?" (id 0) (at 110.49 114.3 0)
+    (property "Reference" "#PWR023" (id 0) (at 110.49 114.3 0)
       (effects (font (size 1.27 1.27)) hide)
     )
@@
   (symbol (lib_id "SN65HVD230DR:SN65HVD230DR") (at 133.35 99.06 0) (unit 1)
     (in_bom yes) (on_board yes) (fields_autoplaced)
-    (property "Reference" "U?" (id 0) (at 133.35 81.534 0))
+    (property "Reference" "U3" (id 0) (at 133.35 81.534 0))
     (property "Value" "SN65HVD230DR" (id 1) (at 133.35 84.074 0))
     (property "Footprint" "SOIC127P599X175-8N" (id 2) (at 133.35 99.06 0)
@@
   (symbol (lib_id "Terminal_Block:282837-2") (at 82.55 97.79 0) (unit 1)
     (in_bom yes) (on_board yes) (fields_autoplaced)
-    (property "Reference" "P?" (id 0) (at 86.36 97.7899 0)
+    (property "Reference" "P2" (id 0) (at 86.36 97.7899 0)
       (effects (font (size 1.27 1.27)) (justify left))
     )

Commit message: Added AMS1117 for ESP32-S3
Changed lines of the file:
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@@
     (effects (font (size 1 1)) (justify left bottom))
-  )
-  (label "3V3" (at 170.18 90.17 270)
-    (effects (font (size 1 1)) (justify right bottom))
-  )
-  (label "3V3" (at 153.67 88.9 180)
-    (effects (font (size 1 1)) (justify right bottom))
   )
   (label "CANL" (at 153.67 96.52 180)
@@
     (effects (font (size 1 1)) (justify left bottom))
   )
-  (global_label "3V3" (shape input) (at 153.67 88.9 0) (fields_autoplaced)
+  (hierarchical_label "3V3" (shape input) (at 153.67 88.9 0)
     (effects (font (size 1 1)) (justify left))
-    (property "Intersheet References" "${INTERSHEET_REFS}" (id 0) (at 158.3319 88.8375 0)
-      (effects (font (size 1 1)) (justify left) hide)
-    )
+  )
+  (hierarchical_label "3V3" (shape input) (at 170.18 90.17 90)
+    (effects (font (size 1 1)) (justify left))
   )
   (hierarchical_label "D" (shape input) (at 113.03 93.98 180)

Commit message: added electrolytic capacitors
Parts:
- C9: footprint (none) -> Capacitor_SMD:C_0603_1608Metric
- P2: footprint TE_282837-2 -> TerminalBlock:TerminalBlock_bornier-2_P5.08mm
- R13: footprint (none) -> Resistor_SMD:R_0603_1608Metric
- U3: footprint SOIC127P599X175-8N -> CAN-BUS-IC:SOIC127P599X175-8N
Changed lines of the file:
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@@
       (effects (font (size 1 1)) (justify left))
     )
-    (property "Footprint" "" (id 2) (at 171.1452 102.87 0)
+    (property "Footprint" "Capacitor_SMD:C_0603_1608Metric" (id 2) (at 171.1452 102.87 0)
       (effects (font (size 1.27 1.27)) hide)
     )
@@
       (effects (font (size 1 1)) (justify left))
     )
-    (property "Footprint" "" (id 2) (at 108.712 102.87 90)
+    (property "Footprint" "Resistor_SMD:R_0603_1608Metric" (id 2) (at 108.712 102.87 90)
       (effects (font (size 1.27 1.27)) hide)
     )
@@
     (property "Reference" "U3" (id 0) (at 133.35 81.534 0))
     (property "Value" "SN65HVD230DR" (id 1) (at 133.35 84.074 0))
-    (property "Footprint" "SOIC127P599X175-8N" (id 2) (at 133.35 99.06 0)
+    (property "Footprint" "CAN-BUS-IC:SOIC127P599X175-8N" (id 2) (at 133.35 99.06 0)
       (effects (font (size 1.27 1.27)) (justify bottom) hide)
     )
@@
       (effects (font (size 1.27 1.27)) (justify left))
     )
-    (property "Footprint" "TE_282837-2" (id 2) (at 82.55 97.79 0)
+    (property "Footprint" "TerminalBlock:TerminalBlock_bornier-2_P5.08mm" (id 2) (at 82.55 97.79 0)
       (effects (font (size 1.27 1.27)) (justify bottom) hide)
     )
