File: PCB_Design/Titan-Legs/CAN_BUS.kicad_sch (KiCad schematic)
At the start: 4 parts, among them P2 282837-2, U3 SN65HVD230DR

Commit message: Added Electrolytic Capacitor and moved AMS1117 to B.Cu
Parts:
- removed C9: 0.1uF, Capacitor_SMD:C_0603_1608Metric, symbol Device:C
- removed P2: 282837-2, TerminalBlock:TerminalBlock_bornier-2_P5.08mm, symbol Terminal_Block:282837-2
- removed R13: 10K, Resistor_SMD:R_0402_1005Metric, symbol Device:R
- removed U3: SN65HVD230DR, CAN-BUS-IC:SOIC127P599X175-8N, symbol SN65HVD230DR:SN65HVD230DR
Connections:
- no-connect marks 1 -> 0
Changed lines of the file:
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@@
 (kicad_sch (version 20211123) (generator eeschema)
   (paper "A4")
-  (junction (at 110.49 96.52) (diameter 0) (color 0 0 0 0)
-  )
-  (no_connect (at 151.13 101.6))
-  (wire (pts (xy 170.18 90.17) (xy 170.18 95.25))
-    (stroke (width 0) (type default) (color 0 0 0 0))
-  )
-  (wire (pts (xy 109.5756 96.52) (xy 110.49 96.52))
-    (stroke (width 0) (type default) (color 0 0 0 0))
-  )
-  (wire (pts (xy 151.13 109.22) (xy 152.4 109.22))
-    (stroke (width 0) (type default) (color 0 0 0 0))
-  )
-  (wire (pts (xy 69.85 97.79) (xy 74.93 97.79))
-    (stroke (width 0) (type default) (color 0 0 0 0))
-  )
-  (wire (pts (xy 151.13 93.98) (xy 153.67 93.98))
-    (stroke (width 0) (type default) (color 0 0 0 0))
-  )
-  (wire (pts (xy 151.13 96.52) (xy 153.67 96.52))
-    (stroke (width 0) (type default) (color 0 0 0 0))
-  )
-  (wire (pts (xy 113.03 93.98) (xy 115.57 93.98))
-    (stroke (width 0) (type default) (color 0 0 0 0))
-  )
-  (wire (pts (xy 151.13 99.06) (xy 153.67 99.06))
-    (stroke (width 0) (type default) (color 0 0 0 0))
-  )
-  (wire (pts (xy 151.13 88.9) (xy 153.67 88.9))
-    (stroke (width 0) (type default) (color 0 0 0 0))
-  )
-  (wire (pts (xy 69.85 100.33) (xy 74.93 100.33))
-    (stroke (width 0) (type default) (color 0 0 0 0))
-  )
-  (wire (pts (xy 110.49 96.52) (xy 115.57 96.52))
-    (stroke (width 0) (type default) (color 0 0 0 0))
-  )
-  (wire (pts (xy 152.4 109.22) (xy 152.4 110.49))
-    (stroke (width 0) (type default) (color 0 0 0 0))
-  )
-  (wire (pts (xy 170.18 102.87) (xy 170.18 105.41))
-    (stroke (width 0) (type default) (color 0 0 0 0))
-  )
-  (wire (pts (xy 110.49 96.52) (xy 110.49 99.06))
-    (stroke (width 0) (type default) (color 0 0 0 0))
-  )
-  (wire (pts (xy 110.49 106.68) (xy 110.49 107.95))
-    (stroke (width 0) (type default) (color 0 0 0 0))
-  )
-  (label "CANH" (at 153.67 93.98 180)
-    (effects (font (size 1 1)) (justify right bottom))
-  )
-  (label "CANL" (at 69.85 100.33 0)
-    (effects (font (size 1 1)) (justify left bottom))
-  )
-  (label "CANL" (at 153.67 96.52 180)
-    (effects (font (size 1 1)) (justify right bottom))
-  )
-  (label "IO35" (at 113.03 96.52 0)
-    (effects (font (size 1 1)) (justify left bottom))
-  )
-  (label "IO17" (at 113.03 93.98 0)
-    (effects (font (size 1 1)) (justify left bottom))
-  )
-  (label "IO18" (at 153.67 99.06 180)
-    (effects (font (size 1 1)) (justify right bottom))
-  )
-  (label "CANH" (at 69.85 97.79 0)
-    (effects (font (size 1 1)) (justify left bottom))
-  )
-  (hierarchical_label "3V3" (shape input) (at 153.67 88.9 0)
-    (effects (font (size 1 1)) (justify left))
-  )
-  (hierarchical_label "3V3" (shape input) (at 170.18 90.17 90)
-    (effects (font (size 1 1)) (justify left))
-  )
-  (hierarchical_label "D" (shape input) (at 113.03 93.98 180)
-    (effects (font (size 1 1)) (justify right))
-  )
-  (hierarchical_label "R" (shape input) (at 153.67 99.06 0)
-    (effects (font (size 1 1)) (justify left))
-  )
-  (hierarchical_label "RS" (shape input) (at 109.5756 96.52 180)
-    (effects (font (size 1 1)) (justify right))
-  )
-  (symbol (lib_id "power:GND") (at 170.18 105.41 0) (unit 1)
-    (in_bom yes) (on_board yes)
-    (property "Reference" "#PWR025" (id 0) (at 170.18 111.76 0)
-      (effects (font (size 1.27 1.27)) hide)
-    )
-    (property "Value" "GND" (id 1) (at 170.434 108.966 0)
-      (effects (font (size 0.762 0.762)))
-    )
-    (property "Footprint" "" (id 2) (at 170.18 105.41 0)
-      (effects (font (size 1.27 1.27)) hide)
-    )
-    (property "Datasheet" "" (id 3) (at 170.18 105.41 0)
-      (effects (font (size 1.27 1.27)) hide)
-    )
-    (pin "1")
-  )
-  (symbol (lib_id "power:GND") (at 152.4 110.49 0) (unit 1)
-    (in_bom yes) (on_board yes) (fields_autoplaced)
-    (property "Reference" "#PWR024" (id 0) (at 152.4 116.84 0)
-      (effects (font (size 1.27 1.27)) hide)
-    )
-    (property "Value" "GND" (id 1) (at 152.4 115.062 0)
-      (effects (font (size 0.762 0.762)))
-    )
-    (property "Footprint" "" (id 2) (at 152.4 110.49 0)
-      (effects (font (size 1.27 1.27)) hide)
-    )
-    (property "Datasheet" "" (id 3) (at 152.4 110.49 0)
-      (effects (font (size 1.27 1.27)) hide)
-    )
-    (pin "1")
-  )
-  (symbol (lib_id "Device:C") (at 170.18 99.06 0) (unit 1)
-    (in_bom yes) (on_board yes)
-    (property "Reference" "C9" (id 0) (at 171.45 96.52 0)
-      (effects (font (size 1 1)) (justify left))
-    )
-    (property "Value" "0.1uF" (id 1) (at 168.91 105.41 90)
-      (effects (font (size 1 1)) (justify left))
-    )
-    (property "Footprint" "Capacitor_SMD:C_0603_1608Metric" (id 2) (at 171.1452 102.87 0)
-      (effects (font (size 1.27 1.27)) hide)
-    )
-    (property "Datasheet" "~" (id 3) (at 170.18 99.06 0)
-      (effects (font (size 1.27 1.27)) hide)
-    )
-    (pin "1")
-    (pin "2")
-  )
-  (symbol (lib_id "Device:R") (at 110.49 102.87 0) (unit 1)
-    (in_bom yes) (on_board yes)
-    (property "Reference" "R13" (id 0) (at 113.03 100.33 0)
-      (effects (font (size 1 1)) (justify left))
-    )
-    (property "Value" "10K" (id 1) (at 110.49 104.14 90)
-      (effects (font (size 1 1)) (justify left))
-    )
-    (property "Footprint" "Resistor_SMD:R_0402_1005Metric" (id 2) (at 108.712 102.87 90)
-      (effects (font (size 1.27 1.27)) hide)
-    )
-    (property "Datasheet" "~" (id 3) (at 110.49 102.87 0)
-      (effects (font (size 1.27 1.27)) hide)
-    )
-    (pin "1")
-    (pin "2")
-  )
-  (symbol (lib_id "power:GND") (at 110.49 107.95 0) (unit 1)
-    (in_bom yes) (on_board yes) (fields_autoplaced)
-    (property "Reference" "#PWR023" (id 0) (at 110.49 114.3 0)
-      (effects (font (size 1.27 1.27)) hide)
-    )
-    (property "Value" "GND" (id 1) (at 110.49 112.522 0)
-      (effects (font (size 0.762 0.762)))
-    )
-    (property "Footprint" "" (id 2) (at 110.49 107.95 0)
-      (effects (font (size 1.27 1.27)) hide)
-    )
-    (property "Datasheet" "" (id 3) (at 110.49 107.95 0)
-      (effects (font (size 1.27 1.27)) hide)
-    )
-    (pin "1")
-  )
-  (symbol (lib_id "SN65HVD230DR:SN65HVD230DR") (at 133.35 99.06 0) (unit 1)
-    (in_bom yes) (on_board yes) (fields_autoplaced)
-    (property "Reference" "U3" (id 0) (at 133.35 81.534 0))
-    (property "Value" "SN65HVD230DR" (id 1) (at 133.35 84.074 0))
-    (property "Footprint" "CAN-BUS-IC:SOIC127P599X175-8N" (id 2) (at 133.35 99.06 0)
-      (effects (font (size 1.27 1.27)) (justify bottom) hide)
-    )
-    (property "Datasheet" "" (id 3) (at 133.35 99.06 0)
-      (effects (font (size 1.27 1.27)) hide)
-    )
-    (pin "1")
-    (pin "2")
-    (pin "3")
-    (pin "4")
-    (pin "5")
-    (pin "6")
-    (pin "7")
-    (pin "8")
-  )
-  (symbol (lib_id "Terminal_Block:282837-2") (at 82.55 97.79 0) (unit 1)
-    (in_bom yes) (on_board yes) (fields_autoplaced)
-    (property "Reference" "P2" (id 0) (at 86.36 97.7899 0)
-      (effects (font (size 1.27 1.27)) (justify left))
-    )
-    (property "Value" "282837-2" (id 1) (at 86.36 100.3299 0)
-      (effects (font (size 1.27 1.27)) (justify left))
-    )
-    (property "Footprint" "TerminalBlock:TerminalBlock_bornier-2_P5.08mm" (id 2) (at 82.55 97.79 0)
-      (effects (font (size 1.27 1.27)) (justify bottom) hide)
-    )
-    (property "Datasheet" "" (id 3) (at 82.55 97.79 0)
-      (effects (font (size 1.27 1.27)) hide)
-    )
-    (property "Comment" "282837-2" (id 4) (at 82.55 97.79 0)
-      (effects (font (size 1.27 1.27)) (justify bottom) hide)
-    )
-    (pin "1")
-    (pin "2")
-  )
 )
