File: PCB_Design/Titan-Legs/DRV8323.kicad_sch (KiCad schematic)
At the start: 26 parts, among them IC3 DRV8323RSRGZT, J2 1986660-3, Q1 BSC031N06NS3GATMA1, Q2 BSC031N06NS3GATMA1, Q3 BSC031N06NS3GATMA1, Q4 BSC031N06NS3GATMA1, Q5 BSC031N06NS3GATMA1, Q6 BSC031N06NS3GATMA1

Commit message: DRV8323 and CP2102 routing initiated
Parts:
- removed J2: 1986660-3, 3x Terminal Block:TE_1986660-3, symbol 3_Pin_Terminal_Block:1986660-3
- added J2: 1546216-3, TB - 3:15462163, symbol TB - 3:1546216-3
- R14, R15, R16: footprint 3x Terminal Block:0.5m_resistor -> Resistor_6.4mm_3.2mm_1.2mm_pads:R_0.5m
Connections:
- net MOTOR_A: now also J2.1
- net MOTOR_B: now also J2.2
- net MOTOR_C: now also J2.3
Changed lines of the file:
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@@
+    (stroke (width 0) (type default) (color 0 0 0 0))
+  )
+  (wire (pts (xy 265.4808 96.5708) (xy 263.4996 96.5708))
     (stroke (width 0) (type default) (color 0 0 0 0))
   )
@@
     (pin "2")
   )
-  (symbol (lib_id "power:GND") (at 263.4996 96.5708 90) (unit 1)
-    (in_bom yes) (on_board yes)
-    (property "Reference" "#PWR038" (id 0) (at 269.8496 96.5708 0)
-      (effects (font (size 1.27 1.27)) hide)
-    )
-    (property "Value" "GND" (id 1) (at 267.3096 96.5708 0)
-      (effects (font (size 1 1)))
-    )
-    (property "Footprint" "" (id 2) (at 263.4996 96.5708 0)
-      (effects (font (size 1.27 1.27)) hide)
-    )
-    (property "Datasheet" "" (id 3) (at 263.4996 96.5708 0)
+  (symbol (lib_id "power:GND") (at 265.4808 96.5708 90) (unit 1)
+    (in_bom yes) (on_board yes)
+    (property "Reference" "#PWR038" (id 0) (at 271.8308 96.5708 0)
+      (effects (font (size 1.27 1.27)) hide)
+    )
+    (property "Value" "GND" (id 1) (at 269.2908 96.5708 0)
+      (effects (font (size 1 1)))
+    )
+    (property "Footprint" "" (id 2) (at 265.4808 96.5708 0)
+      (effects (font (size 1.27 1.27)) hide)
+    )
+    (property "Datasheet" "" (id 3) (at 265.4808 96.5708 0)
       (effects (font (size 1.27 1.27)) hide)
     )
@@
       (effects (font (size 1 1)) (justify left))
     )
-    (property "Footprint" "3x Terminal Block:0.5m_resistor" (id 2) (at 26.162 111.76 90)
+    (property "Footprint" "Resistor_6.4mm_3.2mm_1.2mm_pads:R_0.5m" (id 2) (at 26.162 111.76 90)
       (effects (font (size 1.27 1.27)) hide)
     )
@@
       (effects (font (size 1 1)) (justify left))
     )
-    (property "Footprint" "3x Terminal Block:0.5m_resistor" (id 2) (at 61.722 111.76 90)
+    (property "Footprint" "Resistor_6.4mm_3.2mm_1.2mm_pads:R_0.5m" (id 2) (at 61.722 111.76 90)
       (effects (font (size 1.27 1.27)) hide)
     )
@@
   (symbol (lib_id "Device:R") (at 249.5296 97.3328 0) (unit 1)
     (in_bom yes) (on_board yes)
-    (property "Reference" "R17" (id 0) (at 248.7676 97.0788 0)
+    (property "Reference" "R17" (id 0) (at 249.5296 98.1964 90)
       (effects (font (size 0.762 0.762)) (justify left))
     )
@@
     (pin "1")
     (pin "2")
-  )
-  (symbol (lib_id "3_Pin_Terminal_Block:1986660-3") (at 74.93 179.07 0) (unit 1)
-    (in_bom yes) (on_board yes) (fields_autoplaced)
-    (property "Reference" "J2" (id 0) (at 81.28 177.7999 0)
-      (effects (font (size 1.27 1.27)) (justify left))
-    )
-    (property "Value" "1986660-3" (id 1) (at 81.28 180.3399 0)
-      (effects (font (size 1.27 1.27)) (justify left))
-    )
-    (property "Footprint" "3x Terminal Block:TE_1986660-3" (id 2) (at 74.93 179.07 0)
-      (effects (font (size 1.27 1.27)) (justify bottom) hide)
-    )
-    (property "Datasheet" "" (id 3) (at 74.93 179.07 0)
-      (effects (font (size 1.27 1.27)) hide)
-    )
-    (property "Comment" "1986660-3" (id 4) (at 74.93 179.07 0)
-      (effects (font (size 1.27 1.27)) (justify bottom) hide)
-    )
-    (pin "1_1")
-    (pin "1_2")
-    (pin "2_1")
-    (pin "2_2")
-    (pin "3_1")
-    (pin "3_2")
   )
   (symbol (lib_id "BSC031N06NS3GATMA1:BSC031N06NS3GATMA1") (at 27.94 105.41 90) (unit 1)
@@
     (pin "8")
   )
+  (symbol (lib_id "TB - 3:1546216-3") (at 64.77 176.53 0) (unit 1)
+    (in_bom yes) (on_board yes) (fields_autoplaced)
+    (property "Reference" "J2" (id 0) (at 81.0768 177.7999 0)
+      (effects (font (size 1.27 1.27)) (justify left))
+    )
+    (property "Value" "1546216-3" (id 1) (at 81.0768 180.3399 0)
+      (effects (font (size 1.27 1.27)) (justify left))
+    )
+    (property "Footprint" "TB - 3:15462163" (id 2) (at 81.28 173.99 0)
+      (effects (font (size 1.27 1.27)) (justify left) hide)
+    )
+    (property "Datasheet" "https://www.te.com/commerce/DocumentDelivery/DDEController?Action=srchrtrv&DocNm=1546216&DocType=Customer+Drawing&DocLang=English&DocFormat=pdf&PartCntxt=1546216-3" (id 3) (at 81.28 176.53 0)
+      (effects (font (size 1.27 1.27)) (justify left) hide)
+    )
+    (property "Description" "Fixed Terminal Blocks TERMI-BLOK PCB MNT 90 3P." (id 4) (at 81.28 179.07 0)
+      (effects (font (size 1.27 1.27)) (justify left) hide)
+    )
+    (property "Height" "10.3" (id 5) (at 81.28 181.61 0)
+      (effects (font (size 1.27 1.27)) (justify left) hide)
+    )
+    (property "Manufacturer_Name" "TE Connectivity" (id 6) (at 81.28 184.15 0)
+      (effects (font (size 1.27 1.27)) (justify left) hide)
+    )
+    (property "Manufacturer_Part_Number" "1546216-3" (id 7) (at 81.28 186.69 0)
+      (effects (font (size 1.27 1.27)) (justify left) hide)
+    )
+    (property "Mouser Part Number" "571-1546216-3" (id 8) (at 81.28 189.23 0)
+      (effects (font (size 1.27 1.27)) (justify left) hide)
+    )
+    (property "Mouser Price/Stock" "https://www.mouser.co.uk/ProductDetail/TE-Connectivity/1546216-3?qs=Lxq28tKK6BO7Pspcq1MLxA%3D%3D" (id 9) (at 81.28 191.77 0)
+      (effects (font (size 1.27 1.27)) (justify left) hide)
+    )
+    (property "Arrow Part Number" "1546216-3" (id 10) (at 81.28 194.31 0)
+      (effects (font (size 1.27 1.27)) (justify left) hide)
+    )
+    (property "Arrow Price/Stock" "https://www.arrow.com/en/products/1546216-3/te-connectivity" (id 11) (at 81.28 196.85 0)
+      (effects (font (size 1.27 1.27)) (justify left) hide)
+    )
+    (property "Mouser Testing Part Number" "" (id 12) (at 81.28 199.39 0)
+      (effects (font (size 1.27 1.27)) (justify left) hide)
+    )
+    (property "Mouser Testing Price/Stock" "" (id 13) (at 81.28 201.93 0)
+      (effects (font (size 1.27 1.27)) (justify left) hide)
+    )
+    (pin "1")
+    (pin "2")
+    (pin "3")
+  )
   (symbol (lib_id "power:GND") (at 86.36 50.8 0) (unit 1)
     (in_bom yes) (on_board yes)
@@
       (effects (font (size 1 1)) (justify left))
     )
-    (property "Footprint" "3x Terminal Block:0.5m_resistor" (id 2) (at 98.552 111.76 90)
-      (effects (font (size 1.27 1.27)) hide)
-    )
+    (property "Footprint" "Resistor_6.4mm_3.2mm_1.2mm_pads:R_0.5m" (id 2) (at 98.552 111.76 90)
+      (effects (font (size 1.27 1.27)) hide)
+    )

Commit message: updating recent changes
Parts:
- removed J2: 1546216-3, TB - 3:15462163, symbol TB - 3:1546216-3
- added J2: 691214110003, TerminalBlock:TerminalBlock_bornier-3_P5.08mm, symbol TB_691214110003:691214110003
Connections:
- net MOTOR_A: now also J2.1
- net MOTOR_B: now also J2.2
- net MOTOR_C: now also J2.3
Changed lines of the file:
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@@
     (pin "2")
+  )
+  (symbol (lib_id "TB_691214110003:691214110003") (at 69.85 179.07 270) (unit 1)
+    (in_bom yes) (on_board yes) (fields_autoplaced)
+    (property "Reference" "J2" (id 0) (at 71.12 177.7999 90)
+      (effects (font (size 1.27 1.27)) (justify left))
+    )
+    (property "Value" "691214110003" (id 1) (at 71.12 180.3399 90)
+      (effects (font (size 1.27 1.27)) (justify left))
+    )
+    (property "Footprint" "TerminalBlock:TerminalBlock_bornier-3_P5.08mm" (id 2) (at 69.85 179.07 0)
+      (effects (font (size 1.27 1.27)) (justify bottom) hide)
+    )
+    (property "Datasheet" "" (id 3) (at 69.85 179.07 0)
+      (effects (font (size 1.27 1.27)) hide)
+    )
+    (property "IR-UL" "10A" (id 4) (at 69.85 179.07 0)
+      (effects (font (size 1.27 1.27)) (justify bottom) hide)
+    )
+    (property "WIRE" "24 to 16 (AWG) 0.205 to 1.31 (mm²)" (id 5) (at 69.85 179.07 0)
+      (effects (font (size 1.27 1.27)) (justify bottom) hide)
+    )
+    (property "PART-NUMBER" "691214110003" (id 6) (at 69.85 179.07 0)
+      (effects (font (size 1.27 1.27)) (justify bottom) hide)
+    )
+    (property "MOUNT" "THT" (id 7) (at 69.85 179.07 0)
+      (effects (font (size 1.27 1.27)) (justify bottom) hide)
+    )
+    (property "TYPE" "Horizontal" (id 8) (at 69.85 179.07 0)
+      (effects (font (size 1.27 1.27)) (justify bottom) hide)
+    )
+    (property "DATASHEET-URL" "https://www.we-online.com/catalog/datasheet/691214110003.pdf" (id 9) (at 69.85 179.07 0)
+      (effects (font (size 1.27 1.27)) (justify bottom) hide)
+    )
+    (property "PITCH" "3.5mm" (id 10) (at 69.85 179.07 0)
+      (effects (font (size 1.27 1.27)) (justify bottom) hide)
+    )
+    (property "WORKING-VOLTAGE-UL" "300V (AC)" (id 11) (at 69.85 179.07 0)
+      (effects (font (size 1.27 1.27)) (justify bottom) hide)
+    )
+    (property "PINS" "3" (id 12) (at 69.85 179.07 0)
+      (effects (font (size 1.27 1.27)) (justify bottom) hide)
+    )
+    (pin "1")
+    (pin "2")
+    (pin "3")
   )
   (symbol (lib_id "BSC031N06NS3GATMA1:BSC031N06NS3GATMA1") (at 100.33 71.12 90) (unit 1)
@@
     (pin "8")
   )
-  (symbol (lib_id "TB - 3:1546216-3") (at 64.77 176.53 0) (unit 1)
-    (in_bom yes) (on_board yes) (fields_autoplaced)
-    (property "Reference" "J2" (id 0) (at 81.0768 177.7999 0)
-      (effects (font (size 1.27 1.27)) (justify left))
-    )
-    (property "Value" "1546216-3" (id 1) (at 81.0768 180.3399 0)
-      (effects (font (size 1.27 1.27)) (justify left))
-    )
-    (property "Footprint" "TB - 3:15462163" (id 2) (at 81.28 173.99 0)
-      (effects (font (size 1.27 1.27)) (justify left) hide)
-    )
-    (property "Datasheet" "https://www.te.com/commerce/DocumentDelivery/DDEController?Action=srchrtrv&DocNm=1546216&DocType=Customer+Drawing&DocLang=English&DocFormat=pdf&PartCntxt=1546216-3" (id 3) (at 81.28 176.53 0)
-      (effects (font (size 1.27 1.27)) (justify left) hide)
-    )
-    (property "Description" "Fixed Terminal Blocks TERMI-BLOK PCB MNT 90 3P." (id 4) (at 81.28 179.07 0)
-      (effects (font (size 1.27 1.27)) (justify left) hide)
-    )
-    (property "Height" "10.3" (id 5) (at 81.28 181.61 0)
-      (effects (font (size 1.27 1.27)) (justify left) hide)
-    )
-    (property "Manufacturer_Name" "TE Connectivity" (id 6) (at 81.28 184.15 0)
-      (effects (font (size 1.27 1.27)) (justify left) hide)
-    )
-    (property "Manufacturer_Part_Number" "1546216-3" (id 7) (at 81.28 186.69 0)
-      (effects (font (size 1.27 1.27)) (justify left) hide)
-    )
-    (property "Mouser Part Number" "571-1546216-3" (id 8) (at 81.28 189.23 0)
-      (effects (font (size 1.27 1.27)) (justify left) hide)
-    )
-    (property "Mouser Price/Stock" "https://www.mouser.co.uk/ProductDetail/TE-Connectivity/1546216-3?qs=Lxq28tKK6BO7Pspcq1MLxA%3D%3D" (id 9) (at 81.28 191.77 0)
-      (effects (font (size 1.27 1.27)) (justify left) hide)
-    )
-    (property "Arrow Part Number" "1546216-3" (id 10) (at 81.28 194.31 0)
-      (effects (font (size 1.27 1.27)) (justify left) hide)
-    )
-    (property "Arrow Price/Stock" "https://www.arrow.com/en/products/1546216-3/te-connectivity" (id 11) (at 81.28 196.85 0)
-      (effects (font (size 1.27 1.27)) (justify left) hide)
-    )
-    (property "Mouser Testing Part Number" "" (id 12) (at 81.28 199.39 0)
-      (effects (font (size 1.27 1.27)) (justify left) hide)
-    )
-    (property "Mouser Testing Price/Stock" "" (id 13) (at 81.28 201.93 0)
-      (effects (font (size 1.27 1.27)) (justify left) hide)
-    )
-    (pin "1")
-    (pin "2")
-    (pin "3")
-  )
   (symbol (lib_id "power:GND") (at 86.36 50.8 0) (unit 1)
