File: PCB_Design/Titan-Legs/Quadruped.kicad_sch (KiCad schematic)
At the start: 46 parts, among them IC1 TPS54260DGQR, IC2 CP2102, J1 TYPE-C-31-M-12, P1 282837-2, SW1 SW_Push, SW2 SW_Push, T1 BC847, T2 BC847, U1 ESP32-S3-WROOM-1, U4 AMS1117-3.3

Commit message: DRV8323 and CP2102 routing initiated
Parts:
- D1, D_Zener1: footprint SS34:DIOM7959X265N -> SS34_NEW:DIOM8059X256N
Other:
- note added: "DRV8323RS"
- note removed: "DRV8323RH"
Changed lines of the file:
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@@
     (effects (font (size 3 3) bold) (justify left bottom))
   )
-  (text "DRV8323RH\n\n" (at 114.554 132.08 0)
+  (text "DRV8323RS\n\n" (at 114.554 132.08 0)
     (effects (font (size 3.5 3.5) bold) (justify left bottom))
   )
@@
     (effects (font (size 1 1)) (justify left bottom))
   )
-  (label "D1" (at 271.78 138.43 180)
+  (label "DC1" (at 271.78 138.43 180)
     (effects (font (size 1 1)) (justify right bottom))
   )
@@
     (effects (font (size 1 1)) (justify left bottom))
   )
-  (label "D3" (at 271.78 148.59 180)
+  (label "DC3" (at 271.78 148.59 180)
     (effects (font (size 1 1)) (justify right bottom))
   )
@@
     (effects (font (size 1 1)) (justify left bottom))
   )
-  (label "D2" (at 271.78 140.97 180)
+  (label "DC2" (at 271.78 140.97 180)
     (effects (font (size 1 1)) (justify right bottom))
   )
@@
     (effects (font (size 1 1)) (justify left bottom))
   )
-  (label "D1" (at 170.18 124.46 270)
+  (label "DC1" (at 170.18 124.46 270)
     (effects (font (size 1 1)) (justify right bottom))
   )
@@
     (effects (font (size 1 1)) (justify left bottom))
   )
-  (label "D3" (at 191.77 124.46 270)
+  (label "DC3" (at 191.77 124.46 270)
     (effects (font (size 1 1)) (justify right bottom))
   )
@@
     (effects (font (size 1 1)) (justify right bottom))
   )
-  (label "D2" (at 180.975 124.46 270)
+  (label "DC2" (at 180.975 124.46 270)
     (effects (font (size 1 1)) (justify right bottom))
   )
@@
     (property "Reference" "D1" (id 0) (at 28.194 104.648 0))
     (property "Value" "D" (id 1) (at 27.94 110.744 0))
-    (property "Footprint" "SS34:DIOM7959X265N" (id 2) (at 28.194 108.204 0)
+    (property "Footprint" "SS34_NEW:DIOM8059X256N" (id 2) (at 28.194 108.204 0)
       (effects (font (size 1.27 1.27)) hide)
     )
@@
       (effects (font (size 0.9 0.9)) (justify left))
     )
-    (property "Footprint" "SS34:DIOM7959X265N" (id 2) (at 81.28 163.83 0)
+    (property "Footprint" "SS34_NEW:DIOM8059X256N" (id 2) (at 81.28 163.83 0)
       (effects (font (size 1.27 1.27)) hide)
     )
@@
     )
     (path "/a872eb23-f7b7-4f71-9aa4-4605e4cbbd2b"
-      (reference "D1") (unit 1) (value "D") (footprint "SS34:DIOM7959X265N")
+      (reference "D1") (unit 1) (value "D") (footprint "SS34_NEW:DIOM8059X256N")
     )
     (path "/4baa8b09-ecfb-4dcc-8570-d6fc2395af66"
@@
     )
     (path "/fddf2939-6581-4168-83e6-bfc5e62b7a8a"
-      (reference "D_Zener1") (unit 1) (value "790mV") (footprint "SS34:DIOM7959X265N")
+      (reference "D_Zener1") (unit 1) (value "790mV") (footprint "SS34_NEW:DIOM8059X256N")
     )
     (path "/b23984b5-9f54-4356-8a16-c3212b50a2a0/168619e9-c663-4616-a034-eddd892637d1"
@@
       (reference "J1") (unit 1) (value "TYPE-C-31-M-12") (footprint "usb c:HRO_TYPE-C-31-M-12")
     )
-    (path "/983771df-a9d8-4c95-b2f8-7263116735ed/9cd07df7-0145-436a-ac32-bb079982c303"
-      (reference "J2") (unit 1) (value "1986660-3") (footprint "3x Terminal Block:TE_1986660-3")
+    (path "/983771df-a9d8-4c95-b2f8-7263116735ed/b6301286-c4e8-4c45-84e6-70bfa4923d27"
+      (reference "J2") (unit 1) (value "1546216-3") (footprint "TB - 3:15462163")
     )
     (path "/32bf2d91-ca5e-4e05-87bc-9c7a4f82f965"
@@
     )
     (path "/983771df-a9d8-4c95-b2f8-7263116735ed/1616499b-6a69-425e-b8fa-e342d6d49a89"
-      (reference "R14") (unit 1) (value "0.5m") (footprint "3x Terminal Block:0.5m_resistor")
+      (reference "R14") (unit 1) (value "0.5m") (footprint "Resistor_6.4mm_3.2mm_1.2mm_pads:R_0.5m")
     )
     (path "/983771df-a9d8-4c95-b2f8-7263116735ed/1708bd84-fbd1-43a0-bf47-73fde1f53fcd"
-      (reference "R15") (unit 1) (value "0.5m") (footprint "3x Terminal Block:0.5m_resistor")
+      (reference "R15") (unit 1) (value "0.5m") (footprint "Resistor_6.4mm_3.2mm_1.2mm_pads:R_0.5m")
     )
     (path "/983771df-a9d8-4c95-b2f8-7263116735ed/e776fb65-2a9b-4a83-89c7-138c132d3c1a"
-      (reference "R16") (unit 1) (value "0.5m") (footprint "3x Terminal Block:0.5m_resistor")
+      (reference "R16") (unit 1) (value "0.5m") (footprint "Resistor_6.4mm_3.2mm_1.2mm_pads:R_0.5m")
     )
     (path "/983771df-a9d8-4c95-b2f8-7263116735ed/8a826e4e-2fbc-4ff3-8fa2-79566921b526"

Commit message: updating recent changes
Parts:
- D1, D_Zener1: footprint SS34_NEW:DIOM8059X256N -> Diode_SMD:D_SMB
Changed lines of the file:
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@@
   )
   (symbol (lib_id "CP2102_new:CP2102") (at 229.87 68.58 0) (unit 1)
-    (in_bom yes) (on_board yes) (fields_autoplaced)
+    (in_bom yes) (on_board yes)
     (property "Reference" "IC2" (id 0) (at 262.89 62.0012 0))
-    (property "Value" "CP2102" (id 1) (at 262.89 64.5412 0))
+    (property "Value" "CP2102" (id 1) (at 245.5164 64.3636 0))
     (property "Footprint" "CP2102:QFN50P500X500X100-29N" (id 2) (at 259.08 55.88 0)
       (effects (font (size 1.27 1.27)) (justify left) hide)
@@
     (property "Reference" "D1" (id 0) (at 28.194 104.648 0))
     (property "Value" "D" (id 1) (at 27.94 110.744 0))
-    (property "Footprint" "SS34_NEW:DIOM8059X256N" (id 2) (at 28.194 108.204 0)
+    (property "Footprint" "Diode_SMD:D_SMB" (id 2) (at 28.194 108.204 0)
       (effects (font (size 1.27 1.27)) hide)
     )
@@
       (effects (font (size 0.9 0.9)) (justify left))
     )
-    (property "Footprint" "SS34_NEW:DIOM8059X256N" (id 2) (at 81.28 163.83 0)
+    (property "Footprint" "Diode_SMD:D_SMB" (id 2) (at 81.28 163.83 0)
       (effects (font (size 1.27 1.27)) hide)
     )
@@
     )
   )
-  (sheet (at 13.97 124.206) (size 14.224 6.096) (fields_autoplaced)
+  (sheet (at 13.97 122.5804) (size 19.05 7.7216) (fields_autoplaced)
     (stroke (width 0.1524) (type solid) (color 0 0 0 0))
     (fill (color 0 0 0 0.0000))
-    (property "Sheet name" "Miscellaneous" (id 0) (at 13.97 123.6294 0)
+    (property "Sheet name" "Miscellaneous" (id 0) (at 13.97 122.0038 0)
       (effects (font (size 1 1)) (justify left bottom))
     )
@@
       (reference "#PWR031") (unit 1) (value "GND") (footprint "")
     )
+    (path "/b23984b5-9f54-4356-8a16-c3212b50a2a0/d3b545ad-427d-4143-b793-c05764b9bf4b"
+      (reference "#PWR032") (unit 1) (value "GND") (footprint "")
+    )
     (path "/983771df-a9d8-4c95-b2f8-7263116735ed/07378506-2595-4739-920b-b13951bf4ab8"
       (reference "#PWR033") (unit 1) (value "GND") (footprint "")
@@
     )
     (path "/a872eb23-f7b7-4f71-9aa4-4605e4cbbd2b"
-      (reference "D1") (unit 1) (value "D") (footprint "SS34_NEW:DIOM8059X256N")
+      (reference "D1") (unit 1) (value "D") (footprint "Diode_SMD:D_SMB")
     )
     (path "/4baa8b09-ecfb-4dcc-8570-d6fc2395af66"
@@
     )
     (path "/fddf2939-6581-4168-83e6-bfc5e62b7a8a"
-      (reference "D_Zener1") (unit 1) (value "790mV") (footprint "SS34_NEW:DIOM8059X256N")
+      (reference "D_Zener1") (unit 1) (value "790mV") (footprint "Diode_SMD:D_SMB")
     )
     (path "/b23984b5-9f54-4356-8a16-c3212b50a2a0/168619e9-c663-4616-a034-eddd892637d1"
@@
       (reference "J1") (unit 1) (value "TYPE-C-31-M-12") (footprint "usb c:HRO_TYPE-C-31-M-12")
     )
-    (path "/983771df-a9d8-4c95-b2f8-7263116735ed/b6301286-c4e8-4c45-84e6-70bfa4923d27"
-      (reference "J2") (unit 1) (value "1546216-3") (footprint "TB - 3:15462163")
+    (path "/983771df-a9d8-4c95-b2f8-7263116735ed/746a919e-2f11-486a-a80b-acf27035996c"
+      (reference "J2") (unit 1) (value "691214110003") (footprint "TerminalBlock:TerminalBlock_bornier-3_P5.08mm")
     )
     (path "/32bf2d91-ca5e-4e05-87bc-9c7a4f82f965"
@@
       (reference "R9") (unit 1) (value "10K") (footprint "Resistor_SMD:R_0603_1608Metric")
     )
+    (path "/b23984b5-9f54-4356-8a16-c3212b50a2a0/ca410c7b-44b9-4164-b021-bbf1896d7bc4"
+      (reference "R10") (unit 1) (value "4.7K") (footprint "Resistor_SMD:R_0603_1608Metric")
+    )
     (path "/68a33b1b-c5a4-46e0-8867-0ecbab278f47"
       (reference "R12") (unit 1) (value "5.1k") (footprint "Resistor_SMD:R_0603_1608Metric")
@@
       (reference "U4") (unit 1) (value "AMS1117-3.3") (footprint "AMS1117-3:SOT229P700X180-4N")
     )
-  )
+    (path "/b23984b5-9f54-4356-8a16-c3212b50a2a0/dcf18123-7947-4cff-84e3-a1720bc41cab"
+      (reference "U5") (unit 1) (value "DS18S20Z+") (footprint "Temp-Sensor_DS18S20Z_:DS18S20Z_")
+    )
+  )
