File: PCB_Design/Titan-Legs/untitled.kicad_sch (KiCad schematic)
At the start: 6 parts, among them U5 DS18S20Z+

Commit message: Added Electrolytic Capacitor and moved AMS1117 to B.Cu
Parts:
- removed H1, H2, H3, H4: MountingHole, MountingHole:MountingHole_4mm, symbol Mechanical:MountingHole
- removed R10: 4.7K, Resistor_SMD:R_0603_1608Metric, symbol Device:R
- removed U5: DS18S20Z+, Temp-Sensor_DS18S20Z_:DS18S20Z_, symbol DS18S20Z_:DS18S20Z+
Other:
- note removed: "Mounting Holes"
- note removed: "Temperature Sensor"
Changed lines of the file:
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@@
 (kicad_sch (version 20211123) (generator eeschema)
   (paper "A4")
-  (polyline (pts (xy 95.758 11.938) (xy 95.758 77.1144))
-    (stroke (width 0) (type default) (color 0 0 0 0))
-  )
-  (wire (pts (xy 101.6 64.77) (xy 101.6 67.31))
-    (stroke (width 0) (type default) (color 0 0 0 0))
-  )
-  (wire (pts (xy 101.6 53.34) (xy 101.6 57.15))
-    (stroke (width 0) (type default) (color 0 0 0 0))
-  )
-  (wire (pts (xy 158.75 49.53) (xy 163.83 49.53))
-    (stroke (width 0) (type default) (color 0 0 0 0))
-  )
-  (wire (pts (xy 120.65 54.61) (xy 123.19 54.61))
-    (stroke (width 0) (type default) (color 0 0 0 0))
-  )
-  (wire (pts (xy 158.75 59.69) (xy 163.83 59.69))
-    (stroke (width 0) (type default) (color 0 0 0 0))
-  )
-  (wire (pts (xy 163.83 59.69) (xy 163.83 60.96))
-    (stroke (width 0) (type default) (color 0 0 0 0))
-  )
-  (polyline (pts (xy 12.0904 77.1144) (xy 95.758 77.1144))
-    (stroke (width 0) (type default) (color 0 0 0 0))
-  )
-  (text "Temperature Sensor" (at 114.2492 31.3436 0)
-    (effects (font (size 3.5 3.5) bold) (justify left bottom))
-  )
-  (text "Mounting Holes\n" (at 30.2768 31.0388 0)
-    (effects (font (size 3.5 3.5) bold) (justify left bottom))
-  )
-  (global_label "3V3_IN" (shape input) (at 163.83 49.53 0) (fields_autoplaced)
-    (effects (font (size 1 1)) (justify left))
-    (property "Intersheet References" "${INTERSHEET_REFS}" (id 0) (at 170.7776 49.4675 0)
-      (effects (font (size 1 1)) (justify left) hide)
-    )
-  )
-  (global_label "3V3_IN" (shape input) (at 101.6 53.34 90) (fields_autoplaced)
-    (effects (font (size 1 1)) (justify left))
-    (property "Intersheet References" "${INTERSHEET_REFS}" (id 0) (at 101.5375 46.3924 90)
-      (effects (font (size 1 1)) (justify left) hide)
-    )
-  )
-  (hierarchical_label "IO20" (shape input) (at 101.6 67.31 270)
-    (effects (font (size 1 1)) (justify right))
-  )
-  (hierarchical_label "IO20" (shape input) (at 120.65 54.61 180)
-    (effects (font (size 1 1)) (justify right))
-  )
-  (symbol (lib_id "Mechanical:MountingHole") (at 34.163 43.18 0) (unit 1)
-    (in_bom yes) (on_board yes)
-    (property "Reference" "H1" (id 0) (at 36.703 42.0116 0)
-      (effects (font (size 1.27 1.27)) (justify left))
-    )
-    (property "Value" "MountingHole" (id 1) (at 36.703 44.323 0)
-      (effects (font (size 1.27 1.27)) (justify left))
-    )
-    (property "Footprint" "MountingHole:MountingHole_4mm" (id 2) (at 34.163 43.18 0)
-      (effects (font (size 1.27 1.27)) hide)
-    )
-    (property "Datasheet" "~" (id 3) (at 34.163 43.18 0)
-      (effects (font (size 1.27 1.27)) hide)
-    )
-  )
-  (symbol (lib_id "Mechanical:MountingHole") (at 54.229 54.737 0) (unit 1)
-    (in_bom yes) (on_board yes)
-    (property "Reference" "H3" (id 0) (at 56.769 53.5686 0)
-      (effects (font (size 1.27 1.27)) (justify left))
-    )
-    (property "Value" "MountingHole" (id 1) (at 56.769 55.88 0)
-      (effects (font (size 1.27 1.27)) (justify left))
-    )
-    (property "Footprint" "MountingHole:MountingHole_4mm" (id 2) (at 54.229 54.737 0)
-      (effects (font (size 1.27 1.27)) hide)
-    )
-    (property "Datasheet" "~" (id 3) (at 54.229 54.737 0)
-      (effects (font (size 1.27 1.27)) hide)
-    )
-  )
-  (symbol (lib_id "Mechanical:MountingHole") (at 54.356 42.926 0) (unit 1)
-    (in_bom yes) (on_board yes)
-    (property "Reference" "H4" (id 0) (at 56.896 41.7576 0)
-      (effects (font (size 1.27 1.27)) (justify left))
-    )
-    (property "Value" "MountingHole" (id 1) (at 56.896 44.069 0)
-      (effects (font (size 1.27 1.27)) (justify left))
-    )
-    (property "Footprint" "MountingHole:MountingHole_4mm" (id 2) (at 54.356 42.926 0)
-      (effects (font (size 1.27 1.27)) hide)
-    )
-    (property "Datasheet" "~" (id 3) (at 54.356 42.926 0)
-      (effects (font (size 1.27 1.27)) hide)
-    )
-  )
-  (symbol (lib_id "Device:R") (at 101.6 60.96 0) (unit 1)
-    (in_bom yes) (on_board yes)
-    (property "Reference" "R10" (id 0) (at 103.6828 60.96 90)
-      (effects (font (size 1 1)))
-    )
-    (property "Value" "4.7K" (id 1) (at 101.6 60.96 90)
-      (effects (font (size 1 1)))
-    )
-    (property "Footprint" "Resistor_SMD:R_0603_1608Metric" (id 2) (at 99.822 60.96 90)
-      (effects (font (size 1.27 1.27)) hide)
-    )
-    (property "Datasheet" "~" (id 3) (at 101.6 60.96 0)
-      (effects (font (size 1.27 1.27)) hide)
-    )
-    (pin "1")
-    (pin "2")
-  )
-  (symbol (lib_id "power:GND") (at 163.83 60.96 0) (unit 1)
-    (in_bom yes) (on_board yes)
-    (property "Reference" "#PWR032" (id 0) (at 163.83 67.31 0)
-      (effects (font (size 1.27 1.27)) hide)
-    )
-    (property "Value" "GND" (id 1) (at 163.9316 64.8716 0))
-    (property "Footprint" "" (id 2) (at 163.83 60.96 0)
-      (effects (font (size 1.27 1.27)) hide)
-    )
-    (property "Datasheet" "" (id 3) (at 163.83 60.96 0)
-      (effects (font (size 1.27 1.27)) hide)
-    )
-    (pin "1")
-  )
-  (symbol (lib_id "DS18S20Z_:DS18S20Z+") (at 140.97 54.61 0) (unit 1)
-    (in_bom yes) (on_board yes) (fields_autoplaced)
-    (property "Reference" "U5" (id 0) (at 140.97 41.3512 0))
-    (property "Value" "DS18S20Z+" (id 1) (at 140.97 43.8912 0))
-    (property "Footprint" "Temp-Sensor_DS18S20Z_:DS18S20Z_" (id 2) (at 140.97 54.61 0)
-      (effects (font (size 1.27 1.27)) (justify left bottom) hide)
-    )
-    (property "Datasheet" "" (id 3) (at 140.97 54.61 0)
-      (effects (font (size 1.27 1.27)) (justify left bottom) hide)
-    )
-    (property "PARTREV" "3" (id 4) (at 140.97 54.61 0)
-      (effects (font (size 1.27 1.27)) (justify left bottom) hide)
-    )
-    (property "STANDARD" "IPC7351B" (id 5) (at 140.97 54.61 0)
-      (effects (font (size 1.27 1.27)) (justify left bottom) hide)
-    )
-    (property "MANUFACTURER" "Maxim Integrated" (id 6) (at 140.97 54.61 0)
-      (effects (font (size 1.27 1.27)) (justify left bottom) hide)
-    )
-    (pin "3")
-    (pin "4")
-    (pin "5")
-  )
-  (symbol (lib_id "Mechanical:MountingHole") (at 34.417 54.991 0) (unit 1)
-    (in_bom yes) (on_board yes)
-    (property "Reference" "H2" (id 0) (at 36.957 53.8226 0)
-      (effects (font (size 1.27 1.27)) (justify left))
-    )
-    (property "Value" "MountingHole" (id 1) (at 36.957 56.134 0)
-      (effects (font (size 1.27 1.27)) (justify left))
-    )
-    (property "Footprint" "MountingHole:MountingHole_4mm" (id 2) (at 34.417 54.991 0)
-      (effects (font (size 1.27 1.27)) hide)
-    )
-    (property "Datasheet" "~" (id 3) (at 34.417 54.991 0)
-      (effects (font (size 1.27 1.27)) hide)
-    )
-  )
 )
